Commit message: move_arms modified

File: AlterEgo_Gazebo_Simulator/ego_description/urdf/ego_v2_robot_gazebo.urdf.xacro (robot description, xacro)
@@ -118,4 +118,9 @@
     </collision>
   </link>
+  <!--
+  <gazebo reference="neck">
+    <gravity>0</gravity>
+  </gazebo>
+  -->
   <joint name="base_to_neck" type="fixed">
     <origin rpy="0.0 0.0 0.0" xyz="0 0 0.6985"/>
@@ -158,9 +163,10 @@
   <joint name="rplidar_joint" type="fixed">
     <axis xyz="0 0 0" />
-    <origin xyz="0 0 0.116" rpy="0 0 3.14"/>
+    <!--previous <origin xyz="0 0 0.116" rpy="0 0 3.14"/> -->
+    <origin xyz="0 0 0.132" rpy="0 0 3.14"/>
     <parent link="base_link"/>
     <child link="laser"/>
   </joint>
-   <link name="laser">
+  <link name="laser">
     <collision>
       <origin xyz="0 1 0" rpy="1.5707 0 4.71"/>
@@ -217,4 +223,9 @@
 	</inertial>
     </link>
+  <!--
+  <gazebo reference="${prefix}_shoulder_flange">
+    <gravity>0</gravity>
+  </gazebo>
+  -->
     <link name="${prefix}_shoulder_cube">
       <visual>
@@ -270,4 +281,9 @@
       </inertial>
     </link>
+  <!--
+  <gazebo reference="${prefix}_arm_flage">
+    <gravity>0</gravity>
+  </gazebo>
+  -->
     <link name="${prefix}_arm_cube">
       <visual>
@@ -329,4 +345,9 @@
       </inertial>
     </link>
+  <!--
+  <gazebo reference="${prefix}_elbow_flange">
+    <gravity>0</gravity>
+  </gazebo>
+  -->
     <link name="${prefix}_elbow_cube">
       <visual>
@@ -388,4 +409,9 @@
       </inertial>
     </link>
+  <!--
+  <gazebo reference="${prefix}_forearm_flange">
+    <gravity>0</gravity>
+  </gazebo>
+  -->
     <link name="${prefix}_forearm_cube">
       <visual>
@@ -466,4 +492,9 @@
       </collision>
     </link>
+  <!--
+  <gazebo reference="${prefix}_flange_EE">
+    <gravity>0</gravity>
+  </gazebo>
+  -->
      <xacro:softhands type="${prefix}"
       version = "v2.0_simple"
